Commit message: Add uhvat control [do not tested]

File: uhvat_description/robots/uhvat2fingers.urdf.xacro (robot description, xacro)
@@ -8,6 +8,6 @@
   <xacro:arg name="origin_xyz" default="0 0 0"/>
   <xacro:arg name="origin_rpy" default="0 0 0"/>
-  <link name="world" />
-  <xacro:uhvat name="uhvat" parent="world">
+  <link name="base_gripper_link" />
+  <xacro:uhvat name="uhvat" parent="base_gripper_link">
     <origin xyz="$(arg origin_xyz)" rpy="$(arg origin_rpy)" />
   </xacro:uhvat>

Commit message: Works good with the system

File: uhvat_description/robots/uhvat2fingers.urdf.xacro (robot description, xacro)
@@ -1,5 +1,5 @@
 <?xml version="1.0"?>
 <robot xmlns:xacro="http://www.ros.org/wiki/xacro"
-       name="exo_simple" >
+       name="uhvat1" >
   <xacro:include filename="$(find uhvat_description)/urdf/uhvat.urdf.xacro"/>
   <xacro:include filename="$(find uhvat_description)/controller/ros_controller.urdf.xacro" />
@@ -8,6 +8,6 @@
   <xacro:arg name="origin_xyz" default="0 0 0"/>
   <xacro:arg name="origin_rpy" default="0 0 0"/>
-  <link name="base_gripper_link" />
-  <xacro:uhvat name="uhvat" parent="base_gripper_link">
+  <link name="tool0" />
+  <xacro:uhvat name="uhvat" parent="tool0">
     <origin xyz="$(arg origin_xyz)" rpy="$(arg origin_rpy)" />
   </xacro:uhvat>

File: uhvat_description/urdf/uhvat.urdf.xacro (robot description, xacro)
@@ -43,5 +43,5 @@
       <origin
         xyz="-0.045 -0.035 0"
-        rpy="0 0 ${PI/2}" />
+        rpy="0 0 ${PI}" />
       <parent
         link="${name}_link_0" />
@@ -72,5 +72,5 @@
             scale="0.0013 0.0013 0.002" />
         </geometry>
-        <material name="Grey"/>
+        <material name="Green"/>
       </visual>
     </link>
@@ -79,5 +79,5 @@
       <origin
         xyz="-0.045 0.035 0"
-        rpy="0 0 ${PI/2}" />
+        rpy="0 0 0" />
       <parent
         link="${name}_link_0" />
@@ -108,5 +108,5 @@
             scale="0.0013 0.0013 0.002" />
         </geometry>
-        <material name="Grey"/>
+        <material name="Orange"/>
       </visual>
     </link>
