Commit message: Add collision

File: uhvat_description/urdf/uhvat.urdf.xacro (robot description, xacro)
@@ -38,4 +38,12 @@
         <material name="Grey"/>
       </visual>
+      <collision>
+        <origin xyz="0 0 0" rpy="0 0 0" />
+        <geometry>
+          <mesh
+            filename="package://uhvat_description/meshes/motor_mount.stl"
+            scale="0.001 0.001 0.001" />
+        </geometry>
+      </collision>
     </link>
     <!-- left finger -->
@@ -74,4 +82,12 @@
         <material name="Green"/>
       </visual>
+      <collision>
+        <origin xyz="0.015 0.025 -0.02" rpy="0 0 0" />
+        <geometry>
+          <mesh
+            filename="package://uhvat_description/meshes/festolike_finger.stl"
+            scale="0.0013 0.0013 0.002" />
+        </geometry>
+      </collision>
     </link>
     <!-- right finger -->
@@ -110,4 +126,12 @@
         <material name="Orange"/>
       </visual>
+      <collision>
+        <origin xyz="0.025 0.025 -0.02" rpy="0 0 0" />
+        <geometry>
+          <mesh
+            filename="package://uhvat_description/meshes/festolike_finger.stl"
+            scale="0.0013 0.0013 0.002" />
+        </geometry>
+      </collision>
     </link>
     <!--Extensions -->
